File: Hardware/SparkFun_RFM97CW_Breakout.sch (EAGLE design)
At the start: 22 parts, among them J6 THING_PLUS, J7 U.FL, U4 RFM97CW

Commit message: Add datasheet. Organize repo.
Parts:
- removed J6: THING_PLUS, SparkFun-Boards:THING_PLUS
- added FID3, FID4: FIDUCIAL1X2, SparkFun-Aesthetics:FIDUCIAL1X2
- added R1: 10k, SparkFun-Resistors:10KOHM-0603-1/10W-1%
Connections:
- net !RST!: now also JP3.1, R1.1
- net 3.3V: now also R1.2; no longer J6.3V3
- net DIO5: no longer JP3.1
Other:
- note added: "Antenna length (1/4 wave) 915MHz: 3.07" = 78mm"
- note added: "LoRa Radio 18dBm"
- note removed: "Antenna length (1/4 wave) 915MHz: 3.07" = 78mm 434MHz: 6.47" = 164mm"
- moved on the sheet: C1, C2, J1, J7, U4

Commit message: Adding panel for x02
Parts:
- removed J4: (no value), SparkFun-Connectors:CONN_041X04_NO_SILK
- removed J5: (no value), SparkFun-Connectors:CONN_031X03_NO_SILK
- removed JP8: JUMPER-SMT_2_NO_NO-SILK, SparkFun-Jumpers:JUMPER-SMT_2_NO_NO-SILK
- added JP0, JP1: JUMPER-SMT_2_NO_NO-SILK, SparkFun-Jumpers:JUMPER-SMT_2_NO_NO-SILK
- J2: device SparkFun-Connectors:CONN_031X03_NO_SILK -> SparkFun-Connectors:CONN_09NO_SILK
- J3: device SparkFun-Connectors:CONN_031X03_NO_SILK -> SparkFun-Connectors:CONN_12NO_SILK
- JP2: value JUMPER-SMT_2_NC_TRACE_NO-SILK -> JUMPER-SMT_2_NO_NO-SILK; device SparkFun-Jumpers:JUMPER-SMT_2_NC_TRACE_NO-SILK -> SparkFun-Jumpers:JUMPER-SMT_2_NO_NO-SILK
- JP7: value JUMPER-SMT_2_NO_NO-SILK -> JUMPER-SMT_2_NC_TRACE_NO-SILK; device SparkFun-Jumpers:JUMPER-SMT_2_NO_NO-SILK -> SparkFun-Jumpers:JUMPER-SMT_2_NC_TRACE_NO-SILK
Connections:
- removed net N$10: J5.1, JP7.2
- removed net N$9: J5.2, JP6.2
- new net N$4: J3.5, JP1.2
- new net N$5: J3.4, JP0.2
- new net N$6: J3.7, JP3.2
- net !CS!: now also JP7.1; no longer JP2.1
- net !RST!: now also JP6.1; no longer JP3.1
- net 3.3V: now also J3.1; no longer J3.3
- net DIO0: now also JP0.1; no longer JP8.1
- net DIO1: now also JP1.1; no longer JP6.1
- net DIO2: now also JP2.1; no longer JP7.1
- net DIO3: now also JP3.1; no longer JP5.1
- net DIO5: now also JP5.1
- net GND: now also J3.3; no longer J3.1
- net N$1: now also J3.6, JP2.2; no longer J5.3, JP8.2
- net N$2: now also J2.9, JP6.2; no longer J4.4, JP2.2
- net N$3: now also J2.8, JP7.2; no longer J4.3, JP3.2
- net N$7: now also J3.8; no longer J4.2
- net N$8: now also J3.9; no longer J4.1
- net SCK: now also J3.10; no longer J2.1
- net SDI: now also J3.11; no longer J2.2
- net SDO: now also J3.12; no longer J2.3
Other:
- note added: "x02"
- note removed: "v10"
- moved on the sheet: C1, C2, J1, J7, JP3, JP4, JP5, JP6, R1, U4
